File: KicadPCB/RemoteHF.kicad_pcb (KiCad board)
At the start: 2 copper layers, 203.2 x 130.8 mm, 144 parts, among them J1 IsolatedPower, J10 Transmitter, J11 RX/TX, J2 Raspberry_Pi4, J3 NonIsoPower, J4 SDA100, J5 Yeasu Rotator, J6 ANT1, J7 ANT2, J8 ANT3, J9 ANT4, K1 FRD13501, K2 FRD13501, K3 FRD13501, K4 FRD13501, K5 J107F1CS1212VDC.36, Q1 2N7002E, Q10 2N7002E, Q11 2N7002E, Q12 2N7002E, Q13 2N7002E, Q14 2N7002E, Q15 2N7002E, Q16 2N7002E, Q17 2N7002E, Q18 2N7002E, Q3 2N7002E, Q4 2N7002E, Q5 2N7002E, Q6 2N7002E, Q7 2N7002E, Q8 2N7002E, Q9 2N7002E, U1 MOC8112, U10 MOC8112, U11 MOC8112, U12 MOC8112, U13 MOC8112, U16 MOC8112, U17 MOC8112, U18 MOC8112, U19 MOC8112, U2 MOC8112, U20 MOC8112, U3 MAX232, U4 LM358, U5 ADS1015IDGS, U6 MCP4728, U7 LM358, U8 MOC8112, U9 MOC8112

Commit message: Latest Change August 2023 - PowerSupply
Parts:
- R15: value 15k -> 5.6k
- R16: value 560 -> 1.5k
- R2: value 270 -> 1k
- R25: value 15k -> 10k
- R26: value 560 -> 0
Changed lines of the file:
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@@
         (effects (font (size 1 1) (thickness 0.15)))
     )
-    (fp_text value "560" (at 0 1.65) (layer "F.Fab")
+    (fp_text value "0" (at 0 1.65) (layer "F.Fab")
         (effects (font (size 1 1) (thickness 0.15)))
     )
@@
         (effects (font (size 1 1) (thickness 0.15)))
     )
-    (fp_text value "15k" (at 0 1.65) (layer "F.Fab")
+    (fp_text value "5.6k" (at 0 1.65) (layer "F.Fab")
         (effects (font (size 1 1) (thickness 0.15)))
     )
@@
         (effects (font (size 1 1) (thickness 0.15)))
     )
-    (fp_text value "560" (at -0.635 1.65) (layer "F.Fab")
+    (fp_text value "1.5k" (at -0.635 1.65) (layer "F.Fab")
         (effects (font (size 1 1) (thickness 0.15)))
     )
@@
         (effects (font (size 1 1) (thickness 0.15)))
     )
-    (fp_text value "15k" (at 0 1.65) (layer "F.Fab")
+    (fp_text value "10k" (at 0 1.65) (layer "F.Fab")
         (effects (font (size 1 1) (thickness 0.15)))
     )
@@
         (effects (font (size 1 1) (thickness 0.15)))
     )
-    (fp_text value "270" (at 0 1.65 -270) (layer "F.Fab")
+    (fp_text value "1k" (at 0 1.65 -270) (layer "F.Fab")
         (effects (font (size 1 1) (thickness 0.15)))
     )
