File: KicadPCB/RemoteHF.kicad_sch (KiCad schematic)
At the start: 137 parts, among them J1 IsolatedPower, J10 Transmitter, J11 RX/TX, J2 Raspberry_Pi4, J3 NonIsoPower, J4 SDA100, J5 Yeasu Rotator, J6 ANT1, J7 ANT2, J8 ANT3, J9 ANT4, K1 FRD13501, K2 FRD13501, K3 FRD13501, K4 FRD13501, K5 J107F1CS1212VDC.36, Q1 2N7002E, Q10 2N7002E, Q11 2N7002E, Q12 2N7002E, Q13 2N7002E, Q14 2N7002E, Q15 2N7002E, Q16 2N7002E, Q17 2N7002E, Q18 2N7002E, Q3 2N7002E, Q4 2N7002E, Q5 2N7002E, Q6 2N7002E, Q7 2N7002E, Q8 2N7002E, Q9 2N7002E, U1 MOC8112, U10 MOC8112, U11 MOC8112, U12 MOC8112, U13 MOC8112, U16 MOC8112, U17 MOC8112, U18 MOC8112, U19 MOC8112, U2 MOC8112, U20 MOC8112, U3 MAX232, U4 LM358, U5 ADS1015IDGS, U6 MCP4728, U7 LM358, U8 MOC8112, U9 MOC8112

Commit message: Latest Change August 2023 - PowerSupply
Parts:
- R2: value 270 -> 1k
Changed lines of the file:
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@@
       (effects (font (size 1.27 1.27)) (justify right))
     )
-    (property "Value" "270" (at 7.62 182.499 0)
+    (property "Value" "1k" (at 7.62 182.499 0)
       (effects (font (size 1.27 1.27)) (justify right))
     )
